Commit message: RGBD Camera is set up

File: ur_gripper_description/urdf/ur5_robot.urdf.xacro (robot description, xacro)
@@ -2,10 +2,15 @@
 <robot xmlns:xacro="http://www.ros.org/wiki/xacro"
        name="ur5" >
+  <property name="pi" value="3.14159265" />
   <!-- common stuff -->
   <xacro:include filename="$(find ur_gripper_description)/urdf/common.gazebo.xacro" />
   <!-- ur5 -->
   <xacro:include filename="$(find ur_gripper_description)/urdf/ur5.urdf.xacro" />
+  <!-- robotiq_c_2finger -->
+  <xacro:include filename="$(find ur_gripper_description)/urdf/gripper/robotiq_c2_model_macro.xacro" />
   <!-- arm -->
   <xacro:ur5_robot prefix="" joint_limited="false"/>
+  <!-- gripper -->
+  <xacro:robotiq_c2_model prefix="gripper_"/>
   <link name="world" />
   <joint name="world_joint" type="fixed">
@@ -14,3 +19,8 @@
     <origin xyz="0.0 0.0 0.0" rpy="0.0 0.0 0.0" />
   </joint>
+  <joint name="gripper_joint" type="fixed">
+    <parent link="tool0" />
+    <child link = "gripper_robotiq_85_adapter_link" />
+    <origin xyz="0.0 0.0 0.0" rpy="${pi/2} ${-pi/2} 0.0" />
+  </joint>
 </robot>

Commit message: object detection working; world frame alignment is fine;

File: ur_gripper_description/urdf/ur5_robot.urdf.xacro (robot description, xacro)
@@ -22,5 +22,5 @@
     <parent link="tool0" />
     <child link = "gripper_robotiq_85_adapter_link" />
-    <origin xyz="0.0 0.0 0.0" rpy="${pi/2} ${-pi/2} 0.0" />
+    <origin xyz="0.0 0.0 0.04" rpy="${pi/2} ${-pi/2} 0.0" />
   </joint>
 </robot>

Commit message: object stacking added; multiple object detection using kmeans

File: ur_gripper_description/urdf/ur5_robot.urdf.xacro (robot description, xacro)
@@ -22,5 +22,5 @@
     <parent link="tool0" />
     <child link = "gripper_robotiq_85_adapter_link" />
-    <origin xyz="0.0 0.0 0.04" rpy="${pi/2} ${-pi/2} 0.0" />
+    <origin xyz="0.0 0.0 0.035" rpy="${pi/2} ${-pi/2} 0.0" />
   </joint>
 </robot>
